File: kicad/payloadDorji/payloadDorji.kicad_pcb (KiCad board)
At the start: 2 copper layers, 50 x 80.7 mm, 22 parts, among them J1 Conn_01x01_Pin, J2 Conn_Coaxial, J3 Conn_01x06_Male, U1 LM386

Commit message: payloadDorji add gps and power
Parts:
- removed REF**: MODULE_NUCLEO-L432KC, NUCLEO-L432KC:MODULE_NUCLEO-L432KC
- removed REF**: DORJI_DRA818V, symbols:DORJI_DRA818V
- added AE1: Antenna, PicoAPRS-CustomFootprints:AC30157-01 GNSS Ceramic Chip, B.Cu at (197.6, 91.8)
- added C10: 100n, Capacitor_SMD:C_0402_1005Metric, B.Cu at (175.2, 89.5)
- added C11: DNP, Capacitor_SMD:C_0603_1608Metric, B.Cu at (182.7, 91.5)
- added C12: DNP, Capacitor_SMD:C_0603_1608Metric, B.Cu at (187.6, 91.5)
- added C13: 10p, Capacitor_SMD:C_0603_1608Metric, B.Cu at (199.9, 97.0)
- added C14: 10u, Capacitor_SMD:C_0603_1608Metric, B.Cu at (186.9, 67.6)
- added C8: 10n, Capacitor_SMD:C_0402_1005Metric, B.Cu at (171.2, 62.8)
- added C9: 100n, Capacitor_SMD:C_0402_1005Metric, B.Cu at (173.4, 88.3)
- added J1: PWR, Connector_PinHeader_2.54mm:PinHeader_1x02_P2.54mm_Vertical, F.Cu at (174.9, 63.2)
- added J4: PWR, Connector_PinHeader_2.54mm:PinHeader_1x02_P2.54mm_Vertical, F.Cu at (192.8, 77.4)
- added J5: UART, Connector_PinHeader_2.54mm:PinHeader_1x02_P2.54mm_Vertical, F.Cu at (169.4, 82.5)
- added L4: 2.0n, Inductor_SMD:L_0603_1608Metric, B.Cu at (185.3, 92.2)
- added L5: 1u, Inductor_SMD:L_0603_1608Metric, B.Cu at (176.1, 71.0)
- added R10: 200k, Resistor_SMD:R_0603_1608Metric, B.Cu at (182.5, 74.7)
- added R11: 620, Resistor_SMD:R_0603_1608Metric, B.Cu at (187.0, 75.6)
- added R6: 0, Resistor_SMD:R_0603_1608Metric, B.Cu at (199.9, 86.8)
- added R7: 0, Resistor_SMD:R_0603_1608Metric, B.Cu at (197.7, 86.8)
- added R8: 390, Resistor_SMD:R_0603_1608Metric, B.Cu at (187.0, 71.8)
- added R9: 1.47M, Resistor_SMD:R_0603_1608Metric, B.Cu at (182.5, 71.7)
- added U2: DRA818V, PicoAPRS-CustomFootprints:DORJI_DRA818V, B.Cu at (148.0, 44.8)
- added U3: MAX-M10M-00B, footprints:MOD18_MAX-M10M_UBL, B.Cu at (175.3, 95.6)
- added U4: NUCLEO-L432KC, NUCLEO-L432KC:MODULE_NUCLEO-L432KC, F.Cu at (157.3, 76.9)
- added U5: TPS61023DRLR, footprints:DRL0006A, B.Cu at (179.6, 73.3)
- added U6: AZ1117H-ADJ, Package_TO_SOT_SMD:SOT-223-3_TabPin2, B.Cu at (194.2, 70.6)
Connections:
- J3 pad 2: /PTT -> /H/L
- J3 pad 4: /H/L -> /PTT
Routing:
- net +3.3V: track 5.70 -> 198.0 mm
- net GND: track 5.55 -> 45.9 mm, vias 40 -> 42
- net GPS_UART_TX: track 0.00 -> 38.0 mm
- net +BATT: track 0.00 -> 30.8 mm
- net +5V: track 36.9 -> 67.2 mm
- net /PTT: track 115.1 -> 89.5 mm
- net /H/L: track 89.5 -> 115.1 mm
- net GPS_UART_RX: track 0.00 -> 21.1 mm
- net Net-(U6-ADJ): track 0.00 -> 6.37 mm
- net Net-(U3-RF_IN): track 0.00 -> 4.71 mm
- net Net-(U5-FB): track 0.00 -> 3.86 mm
- net Net-(U5-SW): track 0.00 -> 3.71 mm
- net Net-(C12-Pad2): track 0.00 -> 1.57 mm
Other:
- board size 50 x 80.7 mm -> 79.8 x 79.8 mm

Commit message: no blow up
Parts:
- added C15: 22u, Capacitor_SMD:C_0603_1608Metric, B.Cu at (190.6, 65.1)
- added C16: 22u, Capacitor_SMD:C_0603_1608Metric, B.Cu at (199.6, 71.3)
- added C17: 1u, Capacitor_SMD:C_0603_1608Metric, B.Cu at (126.6, 32.4)
- added C18: 100n, Capacitor_SMD:C_0603_1608Metric, B.Cu at (126.6, 34.0)
- added C19: 10u, Capacitor_SMD:C_0603_1608Metric, B.Cu at (186.6, 78.6)
- C10, C8, C9: footprint Capacitor_SMD:C_0402_1005Metric -> Capacitor_SMD:C_0603_1608Metric
- L5: footprint Inductor_SMD:L_0603_1608Metric -> Inductor_THT:L_Axial_L5.0mm_D3.6mm_P10.00mm_Horizontal_Murata_BL01RN1A2A2
- moved L5 8.92 mm to (174.6, 79.8), turned to 90 degrees
- moved C10 2.28 mm to (172.9, 89.4)
- moved C9 0.90 mm to (174.2, 87.9)
Connections:
- U4 pad CN4_1: +3.3V -> unconnected-(U4B-VIN-PadCN4_1)
Routing:
- net +BATT: track 30.8 -> 35.2 mm
- net GND: track 45.9 -> 49.2 mm
- net +3.3V: track 198.0 -> 200.9 mm
- net Net-(U5-SW): track 3.71 -> 6.49 mm
- net +5V: track 67.2 -> 69.9 mm
