File: kicad/payloadDorji/payloadDorji.kicad_sch (KiCad schematic)
At the start: 54 parts, among them J1 PWR, J2 Conn_Coaxial, J3 Conn_01x06_Male, J4 PWR, J5 UART, J6 PWR, U1 LM386, U2 DRA818V, U3 MAX-M10M-00B, U4 NUCLEO-L432KC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

Commit message: Fix final missing footprints! OK, NOW everything is fixed.
Parts:
- AE1: footprint PicoAPRS-CustomFootprints:AC30157-01 GNSS Ceramic Chip -> picoaprs:AC30157-01 GNSS Ceramic Chip
- U2: footprint PicoAPRS-CustomFootprints:DORJI_DRA818V -> picoaprs:DORJI_DRA818V
- U3: footprint MOD18_MAX-M10M_UBL -> picoaprs:MOD18_MAX-M10M_UBL
- U4: footprint NUCLEO-L432KC:MODULE_NUCLEO-L432KC -> picoaprs:MODULE_NUCLEO-L432KC
Changed lines of the file:
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@@
 			)
 		)
-		(property "Footprint" "NUCLEO-L432KC:MODULE_NUCLEO-L432KC"
+		(property "Footprint" "picoaprs:MODULE_NUCLEO-L432KC"
 			(at 198.12 82.55 0)
 			(effects
@@
 			)
 		)
-		(property "Footprint" "NUCLEO-L432KC:MODULE_NUCLEO-L432KC"
+		(property "Footprint" "picoaprs:MODULE_NUCLEO-L432KC"
 			(at 198.12 130.81 0)
 			(effects
@@
 			)
 		)
-		(property "Footprint" "MOD18_MAX-M10M_UBL"
+		(property "Footprint" "picoaprs:MOD18_MAX-M10M_UBL"
 			(at 127.508 195.834 0)
 			(effects
@@
 			)
 		)
-		(property "Footprint" "PicoAPRS-CustomFootprints:AC30157-01 GNSS Ceramic Chip"
+		(property "Footprint" "picoaprs:AC30157-01 GNSS Ceramic Chip"
 			(at 53.34 203.2 0)
 			(effects
@@
 			)
 		)
-		(property "Footprint" "PicoAPRS-CustomFootprints:DORJI_DRA818V"
+		(property "Footprint" "picoaprs:DORJI_DRA818V"
 			(at 119.38 82.55 0)
 			(effects
