File: kicad/gnss-test/gnss-test.kicad_sch (KiCad schematic)
At the start: 16 parts, among them J1 PWR, J2 EN, J3 UART, Q1 BSS84, Q2 BSS84, U1 MAX-M10M-00B

Commit message: kicad 9.0 updates
Parts:
- C1, C2: footprint Capacitor_SMD:C_0402_1005Metric -> Capacitor_SMD:C_0603_1608Metric
- C3: value 100n -> 1u; footprint Capacitor_SMD:C_0402_1005Metric -> Capacitor_SMD:C_0603_1608Metric
