File: kicad/gnss-test/gnss-test.kicad_pcb (KiCad board)
At the start: 2 copper layers, 17 x 36.5 mm, 16 parts, among them J1 PWR, J2 EN, J3 UART, Q1 BSS84, Q2 BSS84, U1 MAX-M10M-00B

Commit message: ube
Routing:
- net ~{GPS_RTC_PWR_EN}: track 13.9 -> 15.7 mm
- net GND: track 8.33 -> 7.46 mm, vias 119 -> 0

Commit message: GNSS board V2
This new board is a review of the pre existing GNSS circuitry used with the Dorji circuit. Fixed all DRC errors and implemented via snitching compatible with EPL Fab constraints.
Parts:
- removed AE1: Antenna, PicoAPRS-CustomFootprints:AC30157-01 GNSS Ceramic Chip
- moved C3 2.17 mm to (167.3, 78.7)
- moved Q1 2.13 mm to (167.0, 82.0)
Routing:
- net GND: track 7.46 -> 33.8 mm, vias 0 -> 31
- net Net-(C5-Pad2): track 0.00 -> 10.8 mm
- net ~{GPS_PWR_EN}: track 5.19 -> 8.34 mm
- net +3.3V: track 7.73 -> 9.87 mm
- net Net-(Q1-S): track 10.2 -> 8.18 mm
- net Net-(U1-RF_IN): track 3.24 -> 4.78 mm
Other:
- board size 17 x 36.5 mm -> 17.2 x 36.6 mm

Commit message: GNSS V2.1
Fixed footprint of antenna
Parts:
- added AE1: Antenna, PicoAPRS-CustomFootprints:AC30157-01 GNSS Ceramic Chip, F.Cu at (165.2, 54.6)
Routing:
- net GND: track 33.8 -> 21.1 mm
Changed lines of the file:
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@@
+		)
+	)
+	(footprint "PicoAPRS-CustomFootprints:AC30157-01 GNSS Ceramic Chip"
+		(layer "F.Cu")
+		(at 165.16 54.63)
+		(property "Reference" "AE1"
+			(at 0 -3.7 0)
+			(unlocked yes)
+			(layer "F.SilkS")
+			(effects
+				(font
+					(size 1 1)
+					(thickness 0.1)
+				)
+			)
+		)
+		(property "Value" "Antenna"
+			(at 0 4.1 0)
+			(unlocked yes)
+			(layer "F.Fab")
+			(effects
+				(font
+					(size 1 1)
+					(thickness 0.15)
+				)
+			)
+		)
+		(property "Footprint" "PicoAPRS-CustomFootprints:AC30157-01 GNSS Ceramic Chip"
+			(at 0.9 -1.8 0)
+			(unlocked yes)
+			(layer "F.Fab")
+			(hide yes)
+			(effects
+				(font
+					(size 1 1)
+					(thickness 0.15)
+				)
+			)
+		)
+		(property "Datasheet" ""
+			(at 0.9 -1.8 0)
+			(unlocked yes)
+			(layer "F.Fab")
+			(hide yes)
+			(effects
+				(font
+					(size 1 1)
+					(thickness 0.15)
+				)
+			)
+		)
+		(property "Description" "Antenna"
+			(at 0.9 -1.8 0)
+			(unlocked yes)
+			(layer "F.Fab")
+			(hide yes)
+			(effects
+				(font
+					(size 1 1)
+					(thickness 0.15)
+				)
+			)
+		)
+		(attr smd)
+		(fp_line
+			(start -0.5 -0.1)
+			(end 3 -0.1)
+			(stroke
+				(width 1)
+				(type default)
+			)
+			(layer "F.Cu")
+		)
+		(fp_line
+			(start -0.5 2.5)
+			(end -0.5 0)
+			(stroke
+				(width 1)
+				(type default)
+			)
+			(layer "F.Cu")
+		)
+		(fp_line
+			(start 0.2 -2.3)
+			(end -3.1 -2.3)
+			(stroke
+				(width 0.8)
+				(type default)
+			)
+			(layer "F.Cu")
+		)
+		(fp_line
+			(start 1.6 -2.3)
+			(end 3.1 -2.3)
+			(stroke
+				(width 0.8)
+				(type default)
+			)
+			(layer "F.Cu")
+		)
+		(fp_rect
+			(start -3.5 -3)
+			(end 3.5 3)
+			(stroke
+				(width 0.05)
+				(type default)
+			)
+			(fill none)
+			(layer "F.CrtYd")
+		)
+		(fp_text user "${REFERENCE}"
+			(at 0 5.6 0)
+			(unlocked yes)
+			(layer "F.Fab")
+			(effects
+				(font
+					(size 1 1)
+					(thickness 0.15)
+				)
+			)
+		)
+		(pad "1" smd roundrect
+			(at 1.6 -2.3 180)
+			(size 0.8 1)
+			(layers "F.Cu" "F.Paste" "F.Mask")
+			(roundrect_rratio 0.25)
+			(pinfunction "A")
+			(pintype "input")
+			(thermal_bridge_angle 45)
+		)
+		(pad "2" smd roundrect
+			(at 0.2 -2.3 180)
+			(size 0.8 1)
+			(layers "F.Cu" "F.Paste" "F.Mask")
+			(roundrect_rratio 0.25)
+			(thermal_bridge_angle 45)
 		)
 	)
@@
 	)
 	(segment
-		(start 160.96 70.32)
-		(end 167.49 70.32)
-		(width 0.5)
-		(layer "B.Cu")
-		(net 2)
-	)
-	(segment
-		(start 160.5 69.86)
-		(end 160.96 70.32)
-		(width 0.5)
-		(layer "B.Cu")
-		(net 2)
-	)
-	(segment
-		(start 160.5 64.26)
-		(end 160.5 69.86)
-		(width 0.5)
-		(layer "B.Cu")
-		(net 2)
-	)
-	(segment
 		(start 167.49 70.32)
 		(end 167.88 69.93)
@@
 		(start 164.69 58.485)
 		(end 164.69 54.49)
-		(width 0.5)
+		(width 0.8)
 		(layer "F.Cu")
 		(net 20)
@@
 		(start 164.69 54.49)
 		(end 169.755 54.49)
-		(width 0.5)
+		(width 0.8)
 		(layer "F.Cu")
 		(net 20)

Commit message: kicad 9.0 updates
Parts:
- C1, C2: footprint Capacitor_SMD:C_0402_1005Metric -> Capacitor_SMD:C_0603_1608Metric
- C3: value 100n -> 1u; footprint Capacitor_SMD:C_0402_1005Metric -> Capacitor_SMD:C_0603_1608Metric
- moved C2 0.64 mm to (163.8, 79.1)
- moved C3 0.56 mm to (166.7, 78.8)
- moved C1 0.44 mm to (166.2, 77.2)
Routing:
- net GND: track 21.1 -> 16.2 mm
- net Net-(Q1-S): track 8.18 -> 7.41 mm
- net Net-(Q2-S): track 7.54 -> 8.20 mm
Other:
- board size 17.2 x 36.6 mm -> 18.2 x 36.4 mm
