File: kicad/firmware-edition/firmware-edition.kicad_pcb (KiCad board)
At the start: 2 copper layers, 70.4 x 69.4 mm, 104 parts, among them J1 Solar Panel, J10 GPIO, J11 I2C-3V3, J12 GPIO, J14 I2C-5V, J15 SWD, J16 Conn_01x03, J19 Conn_01x01_Pin, J2 BATT, J20 Conn_01x01_Pin, J21 GPIO, J22 3V3, J3 3V3 Sensor Bus, J6 Conn_01x02, J8 GPIO, Q1 BSS84, Q2 BSS84, Q3 BSS84, SW1 BOOT_DFU, SW2 RST, U1 ADP5091, U2 TPS61023DRLR, U3 MAX-M10M-00B, U4 Si4463, U5 STM32U073KCU6, U6 TXS0102VDCTR, Y1 30MHz

Commit message: via stitch updates
Parts:
- SW1, SW2: footprint Button_Switch_SMD:Panasonic_EVQPUJ_EVQPUA -> Button_Switch_SMD:SW_Push_1TS009xxxx-xxxx-xxxx_6x6x5mm
- moved SW2 1.58 mm to (160.9, 86.5)
- moved SW1 1.43 mm to (170.2, 92.9), turned to 90 degrees
- renumbered SPI to J13, 3.3 to J4
Routing:
- net +3.3V: track 246.5 -> 248.5 mm
- net GND: track 87.3 -> 86.2 mm, vias 62 -> 107
- net Net-(U5-PF2-NRST): track 12.4 -> 13.2 mm
- net /USB_D+: track 16.3 -> 17.1 mm
Other:
- board text added: "5V_EN"
- board text removed: "5_EN"

Commit message: Fixed small issues
Parts:
- J16: value Conn_01x03 -> USB_C
Other:
- board text added: "GPIO2"
- board text added: "GPIO3"
Changed lines of the file:
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@@
 			)
 		)
-		(property "Value" "Conn_01x03"
-			(at 2.45 4 180)
+		(property "Value" "USB_C"
+			(at 2.49 2.42 0)
 			(layer "F.SilkS")
 			(effects
@@
 		)
 	)
+	(gr_text "GPIO3"
+		(at 118.97 127.52 0)
+		(layer "F.SilkS")
+		(effects
+			(font
+				(size 0.5 0.5)
+				(thickness 0.1)
+			)
+			(justify left bottom)
+		)
+	)
 	(gr_text "GND"
 		(at 110.56 71.44 90)
@@
 			)
 			(justify left bottom)
+		)
+	)
+	(gr_text "GPIO2"
+		(at 116.17 127.57 0)
+		(layer "F.SilkS")
+		(effects
+			(font
+				(size 0.5 0.5)
+				(thickness 0.1)
+			)
+			(justify left bottom)

Commit message: rev b final JLC
Parts:
- J16: value USB_C -> USB
Routing:
- net GND: vias 107 -> 114
Other:
- board text added: "3V3"
- board text added: "PicoBalloon Tracker COATL Lab @ PSU Rev. B"
- board text added: "SCL SDA"
- board text added: "SWDIO SWCLK"
- board text added: "~{RF_IRQ} ~{RF_EN}"

Commit message: transistors backwards
Parts:
- J16: value USB -> USB_C
- turned Q2 to 180 degrees
Connections:
- C10 pad 1: Net-(Q1-S) -> Net-(Q1-D)
- C11 pad 1: Net-(Q1-S) -> Net-(Q1-D)
- C17 pad 1: Net-(Q2-S) -> Net-(Q2-D)
- Q1 pad 2: Net-(Q1-S) -> +3.3V
- Q1 pad 3: +3.3V -> Net-(Q1-D)
- Q2 pad 2: Net-(Q2-S) -> +3.3V
- Q2 pad 3: +3.3V -> Net-(Q2-D)
- Q3 pad 2: Net-(J3-Pin_1) -> +3.3V
- Q3 pad 3: +3.3V -> Net-(J3-Pin_1)
- U3 pad 6: Net-(Q2-S) -> Net-(Q2-D)
- U3 pad 7: Net-(Q1-S) -> Net-(Q1-D)
- U3 pad 8: Net-(Q1-S) -> Net-(Q1-D)
Routing:
- net Net-(Q1-S): track 11.6 -> 0.00 mm
- net Net-(Q2-D): track 0.00 -> 11.0 mm
- net Net-(Q1-D): track 0.00 -> 9.87 mm
- net Net-(Q2-S): track 8.67 -> 0.00 mm
- net +3.3V: track 248.5 -> 246.1 mm
- net Net-(J3-Pin_1): track 5.41 -> 6.89 mm

Commit message: rev1 not complete
Parts:
- removed C22, C23: 100n, Capacitor_SMD:C_0603_1608Metric
- removed J10, J12, J21, J8: GPIO, Connector_PinHeader_2.54mm:PinHeader_1x02_P2.54mm_Vertical
- removed J11: I2C-3V3, Connector_PinHeader_2.54mm:PinHeader_1x02_P2.54mm_Vertical
- removed J13: SPI, Connector_PinHeader_2.54mm:PinHeader_1x04_P2.54mm_Vertical
- removed J16: USB_C, Connector_PinHeader_2.54mm:PinHeader_1x03_P2.54mm_Vertical
- removed J19, J20: Conn_01x01_Pin, Connector_PinHeader_2.54mm:PinHeader_1x01_P2.54mm_Vertical
- removed J4: Conn_01x04, Connector_PinHeader_2.54mm:PinHeader_1x04_P2.54mm_Vertical
- removed J6: Conn_01x02, Connector_PinHeader_2.54mm:PinHeader_1x02_P2.54mm_Vertical
- removed JP2: PTS, Jumper:SolderJumper-3_P1.3mm_Bridged12_Pad1.0x1.5mm
- added ?: , , F.Cu at (165.5, 90.3)
- added ?: , , F.Cu at (165.5, 91.6)
- added ?: , , F.Cu at (165.5, 87.7)
- added ?: , , F.Cu at (165.5, 89.0)
- added ?: , , F.Cu at (165.5, 86.4)
- added J5: USB_C_Receptacle_USB2.0_16P, Connector_USB:USB_C_Receptacle_Palconn_UTC16-G, F.Cu at (169.8, 99.0)
- added JP3: PTS, Jumper:SolderJumper-2_P1.3mm_Open_TrianglePad1.0x1.5mm, F.Cu at (161.0, 83.1)
- added R18: 0, Resistor_SMD:R_0402_1005Metric, F.Cu at (173.3, 90.6)
- added R19: 5.1k, Resistor_SMD:R_0402_1005Metric, F.Cu at (173.2, 92.8)
- added R23: 5.1k, Resistor_SMD:R_0402_1005Metric, F.Cu at (171.8, 93.3)
- C1, C10, C11, C12, C13, C14, C15, C16, C17, C18, C19, C2, C20, C21, C24, C25, C26, C27, C3, C4, C5, C6, C7, C8, C9, CC1, CF2, CF3, CR1, CR2: footprint Capacitor_SMD:C_0603_1608Metric -> Capacitor_SMD:C_0402_1005Metric
- CF1: value 30p -> 13p; footprint Capacitor_SMD:C_0603_1608Metric -> Capacitor_SMD:C_0402_1005Metric
- J1: footprint Connector_PinSocket_2.54mm:PinSocket_1x02_P2.54mm_Vertical -> Connector_Wire:SolderWire-0.1sqmm_1x02_P3.6mm_D0.4mm_OD1mm
- JP1: value Power Type Select -> PTS; footprint Jumper:SolderJumper-3_P1.3mm_Bridged12_Pad1.0x1.5mm -> Jumper:SolderJumper-2_P1.3mm_Open_TrianglePad1.0x1.5mm
- L3, LF2, LF3, LF4, LR2, Lchk1: footprint Inductor_SMD:L_0603_1608Metric -> Inductor_SMD:L_0402_1005Metric
- LF1: value 39n -> 91n; footprint Inductor_SMD:L_0603_1608Metric -> Inductor_SMD:L_0402_1005Metric
- LR1: value 300n -> 270n; footprint Inductor_SMD:L_0603_1608Metric -> Inductor_SMD:L_0402_1005Metric
- Q1, Q2, Q3: value BSS84 -> GSFW0201; footprint Package_TO_SOT_SMD:SOT-23 -> Package_TO_SOT_SMD:SOT-883
- R1, R10, R11, R12, R13, R17, R2, R20, R21, R22, R25, R26, R3, R4, R5, R6, R7, R8, R9: footprint Resistor_SMD:R_0603_1608Metric -> Resistor_SMD:R_0402_1005Metric
- R14: value 10M -> 1M; footprint Resistor_SMD:R_0603_1608Metric -> Resistor_SMD:R_0402_1005Metric
- R15: value 1.47M -> 510k; footprint Resistor_SMD:R_0603_1608Metric -> Resistor_SMD:R_0402_1005Metric
- R16: value 200k -> 68k; footprint Resistor_SMD:R_0603_1608Metric -> Resistor_SMD:R_0402_1005Metric
- RF1: value 50 -> 51; footprint Resistor_SMD:R_0603_1608Metric -> Resistor_SMD:R_0402_1005Metric
- moved H3 92.8 mm to (89.5, 90.8)
- moved H1 86.3 mm to (89.5, 76.7)
- moved J14 44.4 mm to (132.5, 76.8), turned to 0 degrees
- moved R22 37.8 mm to (162.9, 70.4), turned to 0 degrees
- moved Y1 37.8 mm to (153.5, 94.1)
- moved L2 37.4 mm to (152.5, 80.0), turned to 180 degrees
- moved H4 37.1 mm to (89.5, 97.9)
- moved C4 36.0 mm to (152.7, 78.3)
- moved U2 35.3 mm to (152.6, 81.7)
- moved CR2 35.1 mm to (156.9, 104.1)
- moved C6 35.1 mm to (151.5, 83.6)
- moved R25 35.1 mm to (182.9, 50.8), turned to 0 degrees
- moved R16 34.5 mm to (152.0, 85.9), turned to 0 degrees
- moved R15 34.5 mm to (152.0, 85.0)
- moved C3 34.4 mm to (153.7, 78.3)
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Connections:
- CR1 pad 1: Net-(U4-RXn) -> Net-(U4-RXp)
- CR2 pad 1: Net-(U4-RXp) -> Net-(U4-RXn)
- JP1 pad 2: Net-(JP1-C) -> Net-(JP1-B)
- LR1 pad 1: Net-(U4-RXp) -> Net-(U4-RXn)
- LR1 pad 2: Net-(U4-RXn) -> Net-(U4-RXp)
- LR2 pad 1: Net-(U4-RXn) -> Net-(U4-RXp)
- R10 pad 1: Net-(JP1-C) -> Net-(JP1-B)
- R13 pad 1: Net-(JP2-C) -> Net-(JP3-B)
- R3 pad 1: Net-(JP2-A) -> Net-(JP3-B)
- R6 pad 1: Net-(JP2-A) -> Net-(JP3-B)
- R6 pad 2: Net-(JP1-A) -> Net-(JP1-B)
- R7 pad 1: Net-(JP1-B) -> Net-(JP1-A)
- U1 pad 1: Net-(JP2-A) -> Net-(JP3-B)
- U1 pad 4: Net-(JP1-A) -> Net-(JP1-B)
- U5 pad 14: ~{GPS_RTC_PWR_EN} -> ~{RF_IRQ}
- U5 pad 15: ~{GPS_PWR_EN} -> GPIO0
- U5 pad 25: LLD -> ~{GPS_PWR_EN}
- U5 pad 26: ~{RF_IRQ} -> ~{GPS_RTC_PWR_EN}
- U5 pad 27: ~{RF_EN} -> LLD
- U5 pad 29: GPIO3 -> PGOOD
- U5 pad 30: GPIO2 -> ~{SNSR_EN}
- U5 pad 6: PGOOD -> ~{RF_EN}
- U5 pad 7: ~{SNSR_EN} -> GPIO3
- U5 pad 8: GPIO1 -> GPIO2
- U5 pad 9: GPIO0 -> GPIO1
Routing:
- net +3.3V: track 246.1 -> 87.9 mm, vias 5 -> 9
- net GPIO2: track 136.6 -> 14.0 mm, vias 1 -> 0
- net GPIO3: track 128.3 -> 15.5 mm, vias 1 -> 0
- net ~{CHRGR_EN}: track 101.5 -> 6.23 mm, vias 5 -> 0
- net ~{RF_EN}: track 112.0 -> 18.0 mm, vias 1 -> 0
- net LLD: track 98.3 -> 14.8 mm, vias 4 -> 2
- net ~{RF_IRQ}: track 90.6 -> 7.97 mm, vias 5 -> 0
- net ~{SNSR_EN}: track 74.8 -> 1.45 mm
- net 5V_EN: track 80.7 -> 15.6 mm
- net +5V: track 67.5 -> 26.6 mm, vias 1 -> 2
- net PGOOD: track 45.0 -> 6.89 mm
- net ~{RF_CS}: track 41.2 -> 8.10 mm, vias 1 -> 0
- net MOSI: track 37.6 -> 8.97 mm, vias 1 -> 2
- net VSYS: track 42.6 -> 16.2 mm, vias 1 -> 3
- net GPIO1: track 38.1 -> 12.0 mm, vias 0 -> 2
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Other:
- board size 70.4 x 69.4 mm -> 23.3 x 62.3 mm
- rule pad_to_mask_clearance: 0 -> 0.038
- board text removed: "+ -"
- board text removed: "3.3"
- board text removed: "3V3"
- board text removed: "5V"
- board text removed: "5V_EN"
- board text removed: "BATT"
- board text removed: "GND"
- board text removed: "GPIO0"
- board text removed: "GPIO1"
- board text removed: "GPIO2"
- board text removed: "GPIO3"
- board text removed: "LLD"
- board text removed: "MISO"
- board text removed: "MOSI"
- board text removed: "PicoBalloon Tracker COATL Lab @ PSU Rev. B"
- board text removed: "RFCS"
- board text removed: "SCL"
- board text removed: "SCL SDA"
- board text removed: "SCLK"
- board text removed: "SDA"
- board text removed: "SNSR_EN"
- board text removed: "SOLAR PANEL"
- board text removed: "SWDIO SWCLK"
- board text removed: "VSYS"
- board text removed: "~{RF_IRQ} ~{RF_EN}"

Commit message: rev C(ompact) pre-review
Parts:
- removed ? (x5): , 
- removed C24: 10p, Capacitor_SMD:C_0402_1005Metric
- removed C26, C27: 0.1u, Capacitor_SMD:C_0402_1005Metric
- removed C8, C9: DNP, Capacitor_SMD:C_0402_1005Metric
- removed H1, H2, H3, H4: MountingHole, MountingHole:MountingHole_3.2mm_M3_ISO14580
- removed J14: I2C-5V, Connector_PinHeader_2.54mm:PinHeader_1x02_P2.54mm_Vertical
- removed J22: 3V3, Connector_PinSocket_2.54mm:PinSocket_1x02_P2.54mm_Vertical
- removed L2: 1u, Inductor_SMD:L_0603_1608Metric
- removed L3: 2.0n, Inductor_SMD:L_0402_1005Metric
- removed R14: 1M, Resistor_SMD:R_0402_1005Metric
- removed R15: 510k, Resistor_SMD:R_0402_1005Metric
- removed R16: 68k, Resistor_SMD:R_0402_1005Metric
- removed R25, R26: 0, Resistor_SMD:R_0402_1005Metric
- removed U6: TXS0102VDCTR, TXS0102V:SSOP8_DCT_TEX
- added C22: 1u, Capacitor_SMD:C_0402_1005Metric, F.Cu at (161.8, 96.7)
- added REF**: NPTH Drill Hole 0.7mm, Footprintsv2:NPTH Drill Hole 0.7mm, F.Cu at (165.2, 91.6)
- added REF**: NPTH Drill Hole 0.7mm, Footprintsv2:NPTH Drill Hole 0.7mm, F.Cu at (165.2, 86.4)
- added REF**: NPTH Drill Hole 0.7mm, Footprintsv2:NPTH Drill Hole 0.7mm, F.Cu at (165.2, 90.3)
- added REF**: NPTH Drill Hole 0.7mm, Footprintsv2:NPTH Drill Hole 0.7mm, F.Cu at (165.2, 87.7)
- added REF**: NPTH Drill Hole 0.7mm, Footprintsv2:NPTH Drill Hole 0.7mm, F.Cu at (165.2, 89.0)
- AE1: value Antenna -> Whip; footprint Footprintsv2:AC30157-01 GNSS Ceramic Chip -> Connector_Wire:SolderWirePad_1x01_SMD_1x2mm
- C12: value 2.2u -> 1u
- C3: value 0.1u -> 100n
- C6: value 10u -> 1u
- CF1: value 13p -> 33p
- CR1: value 13p -> 12p
- J1: footprint Connector_Wire:SolderWire-0.1sqmm_1x02_P3.6mm_D0.4mm_OD1mm -> Capacitor_THT:C_Disc_D3.0mm_W1.6mm_P2.50mm
- J2: footprint Connector_PinSocket_2.54mm:PinSocket_1x02_P2.54mm_Vertical -> Capacitor_THT:C_Disc_D3.0mm_W1.6mm_P2.50mm
- J3: value 3V3 Sensor Bus -> Conn_01x10; footprint Connector_PinSocket_2.54mm:PinSocket_1x02_P2.54mm_Vertical -> Footprintsv2:CON_513389873; moved to B.Cu
- LF1: value 91n -> 39n
- LR2: value 150n -> 180n
- RF1: value 51 -> 49.9
- U2: value TPS61023DRLR -> BME680; footprint TPS:DRL0006A -> Package_LGA:Bosch_LGA-8_3x3mm_P0.8mm_ClockwisePinNumbering
- Y1: footprint Crystal:Crystal_SMD_Abracon_ABM3-2Pin_5.0x3.2mm -> Crystal:Crystal_SMD_2520-4Pin_2.5x2.0mm
- moved Q3 33.6 mm to (153.8, 92.2), turned to 90 degrees
- moved J3 29.0 mm to (154.6, 89.8), turned to 180 degrees
- moved J2 29.0 mm to (152.7, 80.3), turned to -90 degrees
- moved J1 23.0 mm to (153.4, 69.4)
- moved AE1 17.5 mm to (161.3, 56.9), turned to 90 degrees
- moved C6 16.6 mm to (164.0, 94.5), turned to -90 degrees
- moved U2 15.7 mm to (161.8, 94.4), turned to 90 degrees
- moved AE2 7.18 mm to (158.0, 108.6)
- moved CC1 6.75 mm to (159.8, 107.8)
- moved LF4 5.06 mm to (158.3, 107.3), turned to 0 degrees
- moved CF2 4.61 mm to (154.6, 105.5), turned to 180 degrees
- moved CF3 4.59 mm to (158.3, 106.4)
- moved R21 3.87 mm to (160.4, 92.0)
- moved LF3 3.46 mm to (156.4, 106.5), turned to 0 degrees
- moved LF2 1.95 mm to (156.4, 105.5), turned to 180 degrees
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Connections:
- net Net-(U4-RXn) renamed /RXN
- net Net-(U4-RXp) renamed /RXP
- C6 pad 1: +5V -> +3.3V
- J3 pad 1: Net-(J3-Pin_1) -> GND
- J3 pad 2: GND -> /3V3_SNSR
- Q3 pad 3: Net-(J3-Pin_1) -> /3V3_SNSR
- R21 pad 2: GPS_SCL -> SCL
- R22 pad 2: GPS_SDA -> SDA
- U2 pad 1: Net-(U2-FB) -> GND
- U2 pad 2: 5V_EN -> +3.3V
- U2 pad 3: VSYS -> SDA
- U2 pad 4: GND -> SCL
- U2 pad 5: Net-(U2-SW) -> GND
- U2 pad 6: +5V -> +3.3V
- U3 pad 11: Net-(U3-RF_IN) -> Net-(AE1-A)
- U3 pad 16: GPS_SDA -> SDA
- U3 pad 17: GPS_SCL -> SCL
- U4 pad 19: GPIO2 -> unconnected-(U4-GPIO2-Pad19)
- U4 pad 20: GPIO3 -> unconnected-(U4-GPIO3-Pad20)
- U5 pad 18: 5V_EN -> SNSR_FLEX1
- U5 pad 19: GPS_SCL -> SCL
- U5 pad 20: GPS_SDA -> SDA
- U5 pad 7: GPIO3 -> SNSR_FLEX2
- U5 pad 8: GPIO2 -> SNSR_FLEX3
- Y1 pad 2: Net-(U4-XOUT) -> GND
Routing:
- net SDA: track 0.00 -> 54.2 mm, vias 0 -> 4
- net SCL: track 0.00 -> 49.0 mm, vias 0 -> 3
- net GPS_SCL: track 46.8 -> 0.00 mm, vias 2 -> 0
- net +3.3V: track 87.9 -> 45.0 mm, vias 9 -> 12
- net GPS_SDA: track 42.3 -> 0.00 mm, vias 3 -> 0
- net +5V: track 26.6 -> 0.00 mm, vias 2 -> 0
- net 5V_EN: track 15.6 -> 0.00 mm, vias 2 -> 0
- net GPIO3: track 15.5 -> 0.00 mm
- net GPIO2: track 14.0 -> 0.00 mm
- net SCLK: track 8.77 -> 21.7 mm, vias 0 -> 1
- net ~{SNSR_EN}: track 1.45 -> 14.1 mm, vias 1 -> 2
- net MISO: track 7.97 -> 20.3 mm
- net MOSI: track 8.97 -> 20.2 mm
- net GND: track 102.3 -> 113.1 mm, vias 35 -> 183
- net SNSR_FLEX1: track 0.00 -> 7.72 mm, vias 0 -> 1
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- added copper zone on In2.Cu, net +3.3V
- added copper zone on In1.Cu, net GND
- added copper zone on In2.Cu, net GND
- added copper zone on F.Cu, net Net-(J2-Pin_1)
Other:
- board size 23.3 x 62.3 mm -> 22.4 x 53.4 mm
- copper layers 2 -> 4
- rule pad_to_mask_clearance: 0.038 -> 0
- board text added: "+"
- board text added: "."
- board text added: "BATT"
- board text added: "PWR"

Commit message: rev C pre-review 2
Routing:
- net GND: track 113.1 -> 112.9 mm, vias 183 -> 186
Other:
- board text added: "COATL @ PSU | PicoTracker Rev. C | July 2025"
Changed lines of the file:
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@@
 		(layer "Edge.Cuts")
 	)
+	(gr_text "COATL @ PSU | PicoTracker\nRev. C | July 2025"
+		(at 163.6 59 0)
+		(layer "B.Mask")
+		(effects
+			(font
+				(size 0.5 0.5)
+				(thickness 0.1)
+				(bold yes)
+			)
+			(justify left bottom mirror)
+		)
+	)
 	(gr_text "+"
 		(at 153.6 80.35 0)
@@
 	)
 	(segment
+		(start 159.542501 69.637499)
+		(end 159.54 69.64)
+		(width 0.2)
+		(layer "F.Cu")
+		(net 1)
+	)
+	(segment
 		(start 158.965 101.41)
 		(end 159.21 101.41)
@@
 	)
 	(segment
-		(start 159.54 69.112936)
-		(end 159.54 69.64)
-		(width 0.2)
-		(layer "F.Cu")
-		(net 1)
-	)
-	(segment
 		(start 154.12 104.77)
 		(end 154.1 104.75)
@@
 	)
 	(segment
-		(start 159.542501 69.110435)
-		(end 159.54 69.112936)
-		(width 0.2)
-		(layer "F.Cu")
-		(net 1)
-	)
-	(segment
-		(start 159.530001 68.66)
-		(end 159.530001 68.880036)
+		(start 173.044753 90.05)
+		(end 171.304753 90.05)
 		(width 0.2)
 		(layer "F.Cu")
@@
 	)
 	(segment
-		(start 173.044753 90.05)
-		(end 171.304753 90.05)
+		(start 159.542501 69.110435)
+		(end 159.542501 69.637499)
 		(width 0.2)
 		(layer "F.Cu")
@@
 	)
 	(via
+		(at 154.7 73)
+		(size 0.6)
+		(drill 0.3)
+		(layers "F.Cu" "B.Cu")
+		(free yes)
+		(net 1)
+	)
+	(via
 		(at 153.2 56.7)
 		(size 0.6)
@@
 	)
 	(via
-		(at 164.1 70.2)
-		(size 0.6)
-		(drill 0.3)
-		(layers "F.Cu" "B.Cu")
-		(free yes)
-		(net 1)
-	)
-	(via
 		(at 155 102.5)
 		(size 0.6)
@@
 	)
 	(via
+		(at 154.7 71)
+		(size 0.6)
+		(drill 0.3)
+		(layers "F.Cu" "B.Cu")
+		(free yes)
+		(net 1)
+	)
+	(via
 		(at 153.3 75.07)
 		(size 0.5)
@@
 	)
 	(via
+		(at 154.7 72)
+		(size 0.6)
+		(drill 0.3)
+		(layers "F.Cu" "B.Cu")
+		(free yes)
+		(net 1)
+	)
+	(via
 		(at 164 97.25)
 		(size 0.6)
@@
 	)
 	(via
+		(at 154.7 74)
+		(size 0.6)
+		(drill 0.3)
+		(layers "F.Cu" "B.Cu")
+		(free yes)
+		(net 1)
+	)
+	(via
 		(at 159.52 101.72)
 		(size 0.5)
@@
 	)
 	(segment
+		(start 160.296527 91.01)
+		(end 159.86 91.01)
+		(width 0.15)
+		(layer "F.Cu")
+		(net 2)
+	)
+	(segment
 		(start 153.93 76.29)
 		(end 153.51 76.29)
@@
 	)
 	(segment
+		(start 160.585873 91.178669)
+		(end 160.465196 91.178669)
+		(width 0.15)
+		(layer "F.Cu")
+		(net 2)
+	)
+	(segment
 		(start 155.0925 76.76)
 		(end 154.4 76.76)
@@
 	)
 	(segment
-		(start 160.296527 91.01)
-		(end 160.593264 91.306737)
-		(width 0.15)
-		(layer "F.Cu")
-		(net 2)
-	)
-	(segment
 		(start 161.12 100.56)
 		(end 160.2 100.56)
@@
 	)
 	(segment
+		(start 160.465196 91.178669)
+		(end 160.296527 91.01)
+		(width 0.15)
+		(layer "F.Cu")
+		(net 2)
+	)
+	(segment
 		(start 153.44 84.13)
 		(end 154.05 84.13)
@@
 	)
 	(segment
-		(start 159.86 91.01)
-		(end 160.296527 91.01)
-		(width 0.15)
-		(layer "F.Cu")
-		(net 2)
-	)
-	(segment
 		(start 160.9825 94.8175)
 		(end 161.8 94)
@@
 	)
 	(via
-		(at 160.593264 91.306737)
+		(at 160.585873 91.178669)
 		(size 0.5)
 		(drill 0.3)
@@
 	)
 	(segment
+		(start 161.314 90.275)
+		(end 161.339 90.25)
+		(width 0.15)
+		(layer "F.Cu")
+		(net 37)
+	)
+	(segment
 		(start 161.339 91.681)
 		(end 161.339 90.66)
@@
 	)
 	(segment
-		(start 161.339 90.66)
+		(start 161.339 90.25)
 		(end 161.339 88.559063)
 		(width 0.2)
@@
 	)
 	(segment
-		(start 161.339 90.66)
-		(end 160.8 90.66)
-		(width 0.15)
-		(layer "F.Cu")
-		(net 37)
-	)
-	(segment
-		(start 160.8 90.66)
-		(end 160.73 90.59)
+		(start 160.75 90.275)
+		(end 161.314 90.275)
 		(width 0.15)
 		(layer "F.Cu")
@@
 		(net 37)
 	)
+	(segment
+		(start 161.339 90.66)
+		(end 161.339 90.25)
+		(width 0.2)
+		(layer "F.Cu")
+		(net 37)
+	)
 	(via
-		(at 160.73 90.59)
+		(at 160.75 90.275)
 		(size 0.5)
 		(drill 0.3)
@@
 	)
 	(segment
-		(start 162.88 69.713232)
-		(end 162.881 69.714232)
-		(width 0.2)
-		(layer "B.Cu")
-		(net 37)
-	)
-	(segment
-		(start 162.881 69.714232)
-		(end 162.881 73.159)
-		(width 0.2)
+		(start 160.249 90.776)
+		(end 157.019611 90.776)
+		(width 0.15)
 		(layer "B.Cu")
 		(net 37)
 	)
 	(segment
-		(start 160.544 90.776)
-		(end 157.019611 90.776)
+		(start 154.959995 88.716384)
+		(end 154.959995 88.230001)
 		(width 0.15)
 		(layer "B.Cu")
@@
 	)
 	(segment
-		(start 157.019611 90.776)
-		(end 154.959995 88.716384)
-		(width 0.15)
+		(start 162.88 69.713232)
+		(end 162.881 69.714232)
+		(width 0.2)
 		(layer "B.Cu")
 		(net 37)
 	)
 	(segment
-		(start 160.73 90.59)
-		(end 160.544 90.776)
-		(width 0.15)
+		(start 162.881 69.714232)
+		(end 162.881 73.159)
+		(width 0.2)
 		(layer "B.Cu")
 		(net 37)
 	)
 	(segment
-		(start 154.959995 88.716384)
-		(end 154.959995 88.230001)
+		(start 160.75 90.275)
+		(end 160.249 90.776)
 		(width 0.15)
 		(layer "B.Cu")
@@
 	)
 	(segment
+		(start 157.019611 90.776)
+		(end 154.959995 88.716384)
+		(width 0.15)
+		(layer "B.Cu")
+		(net 37)
+	)
+	(segment
 		(start 157.28 83.3725)
 		(end 157.28 85.16)
@@
 	)
 	(segment
-		(start 163.340161 86.809069)
-		(end 163.340161 86.749839)
-		(width 0.2)
+		(start 157.858866 87.38)
+		(end 154.797996 87.38)
+		(width 0.15)
 		(layer "B.Cu")
 		(net 46)
 	)
 	(segment
-		(start 162.22 91.13)
-		(end 160.84 89.75)
-		(width 0.15)
+		(start 163.340161 86.809069)
+		(end 163.340161 86.749839)
+		(width 0.2)
 		(layer "B.Cu")
 		(net 46)
@@
 	)
 	(segment
-		(start 160.228866 89.75)
-		(end 157.858866 87.38)
+		(start 162.22 90.925)
+		(end 161.045 89.75)
 		(width 0.15)
 		(layer "B.Cu")
@@
 	)
 	(segment
-		(start 157.858866 87.38)
-		(end 154.797996 87.38)
-		(width 0.15)
+		(start 163.340161 86.749839)
+		(end 163.43 86.66)
+		(width 0.2)
 		(layer "B.Cu")
 		(net 46)
 	)
 	(segment
-		(start 154.797996 87.38)
-		(end 154.559996 87.618)
+		(start 162.22 91.13)
+		(end 162.22 90.925)
 		(width 0.15)
 		(layer "B.Cu")
@@
 	)
 	(segment
-		(start 154.559996 87.618)
-		(end 154.559996 88.230001)
-		(width 0.15)
+		(start 162.314293 87.834937)
+		(end 163.340161 86.809069)
+		(width 0.2)
 		(layer "B.Cu")
 		(net 46)
 	)
 	(segment
-		(start 163.340161 86.749839)
-		(end 163.43 86.66)
-		(width 0.2)
+		(start 160.228866 89.75)
+		(end 157.858866 87.38)
+		(width 0.15)
 		(layer "B.Cu")
 		(net 46)
 	)
 	(segment
-		(start 162.314293 87.834937)
-		(end 163.340161 86.809069)
-		(width 0.2)
+		(start 161.045 89.75)
+		(end 160.228866 89.75)
+		(width 0.15)
 		(layer "B.Cu")
 		(net 46)
@@
 	)
 	(segment
-		(start 160.84 89.75)
-		(end 160.228866 89.75)
+		(start 154.797996 87.38)
+		(end 154.559996 87.618)
+		(width 0.15)
+		(layer "B.Cu")
+		(net 46)
+	)
+	(segment
+		(start 154.559996 87.618)
+		(end 154.559996 88.230001)
 		(width 0.15)
 		(layer "B.Cu")
